File: _saved_playbutton.sch (KiCad schematic (older format))
At the start: 189 parts, among them P1 USB_OTG, P17 DBG_CONN, P3 ESP8266, Q1 Q_PMOS_GSD, SW2 SW_PUSH, SW3 SW_PUSH, SW4 SW_PUSH, U1 74AHC1G125, U2 SAMD21G18, U3 AP2112K-3.3V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

Commit message: Added digikey part(s) No.
Parts:
- U4: Digikey Part No. (none) -> 706-1219-1-ND
Changed lines of the file:
@@
 F 2 "Housings_DFN_QFN:QFN-28-1EP_4x4mm_Pitch0.4mm" H 13300 8500 60  0001 C CNN
 F 3 "" H 13300 8500 60  0000 C CNN
+F 4 "706-1219-1-ND" H 13300 8500 60  0001 C CNN "Digikey Part No."
 	1    13300 8500
 	1    0    0    -1
